Commit message: gazebo extensions added, gazebo launch file added

File: src/robot_description/urdf/bumperbot.urdf.xacro (robot description, xacro)
@@ -1,8 +1,18 @@
 <?xml version="1.0"?>
 <robot name="bumperbot" xmlns:xacro="http://www.ros.org/wiki/xacro">
+    <!-- including xml files-->
+    <xacro:include filename="$(find robot_description)/urdf/bumperbot_gazebo.xacro" />
     <!-- Define the robot's links and joints -->
     <!-- Parent link -->
     <link name="world"/>
+    <!-- collisions and inertials are important for physics simulation -->
     <link name="base_link">
+        <inertial>
+            <origin xyz="0 0 0.04" rpy="0.0 0.25 0.3"/>
+            <mass value="8.2573504e-01"/>
+            <inertia ixx="2.2124416e-02" ixy="-1.2294101e-04" ixz="3.4938785e-04"
+                     iyy="2.1193702e-02" iyz="-5.0120904e-05"
+                     izz="2.0064271e-02"/>
+        </inertial>
         <visual>
             <origin xyz="0 0 0" rpy="0 0 0"/>
@@ -14,6 +24,19 @@
             </material>
         </visual>
+        <collision>
+            <origin xyz="0 0 0" rpy="0 0 0"/>
+            <geometry>
+                <mesh filename="package://robot_description/meshes/base_link.STL"/>
+            </geometry>
+        </collision>
     </link>
     <link name="wheel_right_link">
+        <inertial>
+            <origin xyz="0 -0.014 0" rpy="0 0 0"/>
+            <mass value="0.0530086090966721"/>
+            <inertia ixx="1.88176298336665E-05" ixy="-4.8444933029987E-10" ixz="1.88163708851143E-08"
+                     iyy="3.11510738647764E-05" iyz="-6.93560663069607E-11"
+                     izz="1.8801969558182E-05"/>
+        </inertial>
         <visual>
             <origin xyz="0 0 0" rpy="1.57 0 0"/>
@@ -25,6 +48,19 @@
             </material>
         </visual>
+        <collision>
+            <origin xyz="0 -0.015 0" rpy="1.57 0 0"/>
+            <geometry>
+                <sphere radius="0.033"/>
+            </geometry>
+        </collision>
     </link>
     <link name="wheel_left_link">
+        <inertial>
+            <origin xyz="0 0.014 0" rpy="0 0 0"/>
+            <mass value="0.0530086043217644"/>
+            <inertia ixx="1.8792911368909E-05" ixy="3.31256392204584E-10" ixz="-1.14082001662767E-08"
+                     iyy="3.11510738759073E-05" iyz="-3.60499245082192E-10"
+                      izz="1.88266886146847E-05"/>
+        </inertial>
         <visual>
             <origin xyz="0 0 0" rpy="-1.57 0 0"/>
@@ -36,6 +72,19 @@
             </material>
         </visual>
+        <collision>
+            <origin xyz="0 0.015 0" rpy="1.57 0 0"/>
+            <geometry>
+                <sphere radius="0.033"/>
+            </geometry>
+        </collision>
     </link>
     <link name="caster_front_link">
+        <inertial>
+            <origin xyz="3.89968128948481E-07 2.40073004698083E-07 0.00219173397061506" rpy="0 0 0"/>
+            <mass value="1.44379265037903E-06"/>
+            <inertia ixx="7.23075276010246E-11" ixy="-6.10956883467859E-16" ixz="2.22849693525031E-15"
+                     iyy="3.8713793085917E-11" iyz="2.93909858781952E-15"
+                     izz="1.00967486676306E-10"/>
+        </inertial>
         <visual>
             <origin xyz="0 0 0" rpy="0 0 0"/>
@@ -47,6 +96,19 @@
             </material>
         </visual>
+        <collision>
+            <origin xyz="0 0 0" rpy="0 0 0"/>
+            <geometry>
+                <sphere radius="0.005"/>
+            </geometry>
+        </collision>
     </link>
     <link name="caster_rear_link">
+        <inertial>
+            <origin xyz="3.8996812895542E-07 2.40073004698083E-07 0.00219173397061509" rpy="0 0 0"/>
+            <mass value="1.44379265037902E-06"/>
+            <inertia ixx="7.23075276010246E-11" ixy="-6.10956872363424E-16" ixz="2.22849693527207E-15"
+                     iyy="3.87137930859167E-11" iyz="2.939098587861E-15"
+                     izz="1.00967486676306E-10"/>
+        </inertial>
         <visual>
             <origin xyz="0 0 0" rpy="0 0 0"/>
@@ -55,4 +117,21 @@
             </geometry>
             <material name="yellow">
+                <color rgba="1 1 0 1"/>
+            </material>
+        </visual>
+        <collision>
+            <origin xyz="0 0 0" rpy="0 0 0"/>
+            <geometry>
+                <sphere radius="0.005"/>
+            </geometry>
+        </collision>
+    </link>
+    <link name="can_link">
+        <visual>
+            <origin xyz="0 0 0" rpy="0 0 0"/>
+            <geometry>
+                <mesh filename="package://robot_description/meshes/can.STL"/>
+            </geometry>
+            <material name="orange">
                 <color rgba="1 1 0 1"/>
             </material>
@@ -69,5 +148,5 @@
         <parent link="base_link"/>
         <child link="wheel_right_link"/>
-        <origin xyz="0 -0.077 0" rpy="0 0 0"/>
+        <origin xyz="0 -0.0701101849418637 0" rpy="0 0 0"/>
         <axis xyz="0 1 0"/>         <!-- The axis of rotation for the wheel around Y-axis -->
     </joint>
@@ -75,5 +154,5 @@
         <parent link="base_link"/>
         <child link="wheel_left_link"/>
-        <origin xyz="0 0.077 0" rpy="0 0 0"/>
+        <origin xyz="0 0.0701101849418642 0" rpy="0 0 0"/>
         <axis xyz="0 1 0"/>         <!-- The axis of rotation for the wheel around Y-axis -->
     </joint>
@@ -89,3 +168,9 @@
         <origin xyz="-0.04755 0 -0.027" rpy="0 0 0"/>
     </joint>
+    <!-- Define the joint connecting the can_link to the base_link -->
+    <joint name="can_joint" type="fixed">
+        <parent link="base_link"/>
+        <child link="can_link"/>
+        <origin xyz="-0.03 0.03 0.078" rpy="1.57 0 0" />
+    </joint>
 </robot>

Commit message: kinematics (translation and rotation matrix from turtlesim)

File: src/robot_description/urdf/bumperbot.urdf.xacro (robot description, xacro)
@@ -9,5 +9,5 @@
     <!-- Define the robot's links and joints -->
     <!-- Parent link -->
-    <link name="world"/>
+    <link name="base_footprint"/>
     <!-- collisions and inertials are important for physics simulation -->
     <link name="base_link">
@@ -144,5 +144,5 @@
     <!-- Define the joint connecting the base_link to the world -->
     <joint name="base_joint" type="fixed">
-        <parent link="world"/>
+        <parent link="base_footprint"/>
         <child link="base_link"/>
         <origin xyz="0 0 0.033" rpy="0 0 0"/>

File: src/robot_description/urdf/bumperbot_gazebo.xacro (robot description, xacro)
@@ -3,21 +3,21 @@
     <!-- Friction coefficients: To avoid slipping of the wheels -->
     <gazebo reference = "wheel_right_link">
-        <mu1>1000000000000.0</mu1>
-        <mu2>1000000000000.0</mu2>
-        <kp>1000000000000.0</kp>
-        <kd>1000000000000.0</kd>
+        <mu1>1.0</mu1>
+        <mu2>1.0</mu2>
+        <kp>1000000.0</kp>
+        <kd>100.0</kd>
         <minDepth>0.001</minDepth>
         <maxVel>0.1</maxVel>
-        <fdir1>1 0 0</fdir1> <!-- indicates the direction of rotation of
+        <!-- <fdir1>1 0 0</fdir1> --> <!-- indicates the direction of rotation of
                                   wheel only for the wheels which can be accuated-->
     </gazebo>
     <gazebo reference = "wheel_left_link">
-        <mu1>1000000000000.0</mu1>
-        <mu2>1000000000000.0</mu2>
-        <kp>1000000000000.0</kp>
-        <kd>1000000000000.0</kd>
+         <mu1>1.0</mu1>
+        <mu2>1.0</mu2>
+        <kp>1000000.0</kp>
+        <kd>100.0</kd>
         <minDepth>0.001</minDepth>
         <maxVel>0.1</maxVel>
-        <fdir1>1 0 0</fdir1> <!-- indicates the direction of rotation of
+        <!-- <fdir1>1 0 0</fdir1> --> <!-- indicates the direction of rotation of
                                   wheel only for the wheels which can be accuated-->
     </gazebo>

Commit message: IMU sensor added in robot urdfand gz_ros2_bridge message added in launch file

File: src/robot_description/urdf/bumperbot.urdf.xacro (robot description, xacro)
@@ -7,4 +7,6 @@
     <!-- including ROS2 Control-->
     <xacro:include filename="$(find robot_description)/urdf/bumperbot_ros2_control.xacro" />
+    <!-- IMU sensor -->
+    <xacro:include filename="$(find robot_description)/urdf/IMU.xacro"/>
     <!-- Define the robot's links and joints -->
     <!-- Parent link -->
@@ -142,4 +144,32 @@
         </visual>
     </link>
+    <!-- adding IMU link -->
+    <link name="imu_link">
+        <inertial>
+            <origin xyz="-0.00552433659106688 0.000168210391520346 0.000514000497342681" rpy="0 0 0"/>
+            <mass value="0.000528415362211671"/>
+            <inertia ixx="1.46176048428261E-08" ixy="1.40015117949421E-10" ixz="-1.99633872937403E-12"
+                     iyy="8.59662482954888E-09" iyz="7.52375112767959E-12"
+                     izz="2.30279421279312E-08" />
+        </inertial>
+        <visual>
+            <origin xyz="0 0 0" rpy="0 0 0"/>
+            <geometry>
+                <mesh filename="package://robot_description/meshes/imu_link.STL"/>
+            </geometry>
+            <material name="yellow">
+                <color rgba="1 1 0 1"/>
+            </material>
+        </visual>
+        <collision>
+            <origin xyz="0 0 0" rpy="0 0 0"/>
+            <geometry>
+                <mesh filename="package://robot_description/meshes/imu_link.STL"/>
+            </geometry>
+            <material name="yellow">
+                <color rgba="1 1 0 1"/>
+            </material>
+        </collision>
+    </link>
     <!-- Define the joint connecting the base_link to the world -->
     <joint name="base_joint" type="fixed">
@@ -178,3 +208,10 @@
         <origin xyz="-0.03 0.03 0.078" rpy="1.57 0 0" />
     </joint>
+    <!-- Define the joint connecting the imu_link to the base_link -->
+    <joint name="imu_joint" type="fixed">
+        <parent link="base_link"/>
+        <child link="imu_link"/>
+        <origin xyz="0 0 0.07" rpy="0 0 0"/>
+        <axis xyz="0 0 0"/>
+    </joint>
 </robot>

File: src/robot_description/urdf/bumperbot_gazebo.xacro (robot description, xacro)
@@ -38,17 +38,27 @@
         <maxVel>0.1</maxVel>
     </gazebo>
-    <!-- For ROS2 CONTROLLER-->
+    <!-- ROS 2 Control and IMU system -->
     <gazebo>
         <!-- ROS 2 Humble -->
         <xacro:if value="$(arg is_ignition)">
-            <plugin filename="ign_ros2_control-system" name="ign_ros2_control::IgnitionROS2ControlPlugin">
-                <parameters>$(find bumperbot_controller)/config/bumperbot_controllers.yaml</parameters> <!-- Add the controller yaml file-->
+            <plugin
+                filename="ign_ros2_control-system"
+                name="ign_ros2_control::IgnitionROS2ControlPlugin">
+                <parameters>$(find bumperbot_controller)/config/bumperbot_controllers.yaml</parameters>
             </plugin>
+            <plugin
+                filename="ignition-gazebo-imu-system"
+                name="ignition::gazebo::systems::Imu"/>
         </xacro:if>
-        <!-- ROS 2 Iron or above -->
+        <!-- ROS 2 Jazzy / Gazebo Harmonic -->
         <xacro:unless value="$(arg is_ignition)">
-            <plugin filename="gz_ros2_control-system" name="gz_ros2_control::GazeboSimROS2ControlPlugin">
-                <parameters>$(find bumperbot_controller)/config/bumperbot_controllers.yaml</parameters> <!-- Add the controller yaml file-->
+            <plugin
+                filename="gz_ros2_control-system"
+                name="gz_ros2_control::GazeboSimROS2ControlPlugin">
+                <parameters>$(find bumperbot_controller)/config/bumperbot_controllers.yaml</parameters>
             </plugin>
+            <plugin
+                filename="gz-sim-imu-system"
+                name="gz::sim::systems::Imu"/>
         </xacro:unless>
     </gazebo>
